Commit message: update

File: urdf/mecanum_bot.urdf.xacro (robot description, xacro)
@@ -2,4 +2,5 @@
 <robot xmlns:xacro="http://www.ros.org/wiki/xacro" name="mecanum_bot">
   <xacro:arg name="controllers_yaml" default=""/>
+  <xacro:arg name="ros2_control_params" default=""/>
   <xacro:property name="PI" value="3.1415926535897931"/>
   <!-- Dimensions -->
@@ -120,4 +121,6 @@
       <origin xyz="${x} ${y} ${body_z/2 - wheel_r}" rpy="0 0 0"/>
       <axis xyz="0 1 0"/>
+      <limit effort="200.0" velocity="100.0"/>
+      <dynamics damping="0.1" friction="0.0"/>
     </joint>
     <xacro:roller parent="${name}" idx="0" angle="0" sign="${roller_sign}"/>
@@ -209,8 +212,19 @@
   <!-- gz_ros2_control plugin: reads robot_description from robot_state_publisher and loads controllers.yaml -->
   <gazebo>
-    <plugin filename="gz_ros2_control-system" name="gz_ros2_control::GazeboSimROS2ControlPlugin">
+    <plugin filename="ign_ros2_control-system" name="ign_ros2_control::IgnitionROS2ControlPlugin">
       <robot_param>robot_description</robot_param>
       <robot_param_node>robot_state_publisher</robot_param_node>
-      <parameters>$(arg controllers_yaml)</parameters>
+      <parameters>$(arg ros2_control_params)</parameters>
+    </plugin>
+  </gazebo>
+  <!-- Gazebo ground-truth pose publisher -->
+  <gazebo>
+    <plugin filename="ignition-gazebo-pose-publisher-system" name="ignition::gazebo::systems::PosePublisher">
+      <publish_model_pose>true</publish_model_pose>
+      <publish_link_pose>false</publish_link_pose>
+      <publish_collision_pose>false</publish_collision_pose>
+      <publish_visual_pose>false</publish_visual_pose>
+      <publish_nested_model_pose>false</publish_nested_model_pose>
+      <use_pose_vector_msg>true</use_pose_vector_msg>
     </plugin>
   </gazebo>
